File: Power-Secondary.kicad_pcb (KiCad board)
At the start: 2 copper layers, 82 x 66 mm, 37 parts, among them J1 SUPP PWR MON, J2 SUPP PWR 1, J3 SUPP PWR 2, J4 DCDC SUPPLY, J5 FUSE OUT, J6 SUPP OUT, J7 LV ENABLE, Q1 S1G1D2S2G2D1, Q1A1 IRFU5305PbF, Q1A2 IRFU5305PbF, Q1A3 IRFU5305PbF, Q1A4 IRFU5305PbF, Q2 S1G1D2S2G2D1, Q3 FDD86250-F085

Commit message: Designed PCB layout for new Power Board
Parts:
- removed D1: 10V, UTSVT_PowerSupp:SOD2512X110N
- removed Q3: FDD86250-F085, UTSVT_PowerSupp:FDD13AN06A0F085
- added C4: 100uF, Capacitor_SMD:C_0805_2012Metric, F.Cu at (119.1, 102.8)
- added F2: Fuse, Fuse:Fuseholder_Blade_Mini_Keystone_3568, F.Cu at (150.1, 64.5)
- added R5: 300k, Resistor_SMD:R_0805_2012Metric, B.Cu at (126.7, 75.2)
- added R6: 100k, Resistor_SMD:R_0805_2012Metric, B.Cu at (126.7, 78.8)
- added R7: 100k, Resistor_SMD:R_0805_2012Metric, F.Cu at (112.8, 98.2)
- added R8: 100k, Resistor_SMD:R_0805_2012Metric, F.Cu at (119.1, 98.7)
- added U1: Nucleo_L432KC, UTSVT_Special:NucleoL432KC, F.Cu at (130.9, 77.4)
- J1: value SUPP PWR MON -> SUPP PWR 1; footprint Connector_Molex:Molex_Micro-Fit_3.0_43650-0215_1x02_P3.00mm_Vertical -> Connector_Molex:Molex_Sabre_43160-0102_1x02_P7.49mm_Vertical
- J2: value SUPP PWR 1 -> SUPP PWR 2
- J3: value SUPP PWR 2 -> SUPP OUT; footprint Connector_Molex:Molex_Sabre_43160-0102_1x02_P7.49mm_Vertical -> Connector_Molex:Molex_Micro-Fit_3.0_43650-0215_1x02_P3.00mm_Vertical
- J4: value DCDC SUPPLY -> SUPP PWR MON; footprint Connector_Molex:Molex_Sabre_43160-0102_1x02_P7.49mm_Vertical -> Connector_Molex:Molex_Micro-Fit_3.0_43650-0215_1x02_P3.00mm_Vertical
- J5: value FUSE OUT -> DCDC SUPPLY
- J6: value SUPP OUT -> LV ENABLE
- J7: value LV ENABLE -> FUSE OUT; footprint Connector_Molex:Molex_Micro-Fit_3.0_43650-0215_1x02_P3.00mm_Vertical -> Connector_Molex:Molex_Sabre_43160-0102_1x02_P7.49mm_Vertical
- LOGO1, LOGO2: moved to F.Cu
- Q1: value S1G1D2S2G2D1 -> FDD86250-F085; footprint UTSVT_PowerSupp:SOT65P210X100-6N -> UTSVT_PowerSupp:FDD13AN06A0F085
- R2: value 10k -> 100k; footprint Resistor_SMD:R_0603_1608Metric -> Resistor_SMD:R_0805_2012Metric
- R3: value 1M -> 5.1K; footprint Resistor_SMD:R_0603_1608Metric -> Resistor_SMD:R_0805_2012Metric
- R4: value 5.1K -> 100k
- TP2: value DCDC_PWR -> DCDC_Gate
- TP3: value ZENER_GATE -> DCDC_PWR
- TP4: value DCDC_Gate -> Supp_Gate
- TP5: value Supp_Gate -> GND
- moved LOGO2 247.1 mm to (-92.1, 106.2), turned to 0 degrees
- moved LOGO1 200.0 mm to (-75.7, 104.8), turned to 0 degrees
- moved H3 72.0 mm to (93.0, 104.0)
- moved H4 72.0 mm to (165.0, 104.0)
- moved J4 50.9 mm to (106.0, 48.0), turned to 0 degrees
- moved R4 38.9 mm to (106.1, 62.9), turned to -90 degrees
- moved Q2 37.2 mm to (115.9, 98.5)
- moved J1 30.7 mm to (100.5, 67.5), turned to 90 degrees
- moved Q1 30.7 mm to (147.5, 90.0), turned to 0 degrees
- moved J6 28.1 mm to (148.0, 104.0)
- moved Q1A2 27.1 mm to (110.8, 69.5), turned to 0 degrees
- moved Q1A4 27.1 mm to (110.8, 63.9), turned to 0 degrees
- moved TP2 25.1 mm to (118.3, 48.0)
- moved J2 24.1 mm to (100.5, 91.5)
- moved J5 24.1 mm to (157.0, 60.0)
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Connections:
- F1 pad 1: Net-(F1-Pad1) -> Net-(J1-Pin_1)
- F1 pad 2: FUSE_OUT -> SUPP_PWR
- J1 pad 1: SUPP_PWR -> Net-(J1-Pin_1)
- J2 pad 1: SUPP_PWR -> Net-(J1-Pin_1)
- J3 pad 1: SUPP_PWR -> Net-(J1-Pin_1)
- J4 pad 1: DCDC_PWR -> Net-(J1-Pin_1)
- J5 pad 1: FUSE_OUT -> DCDC_PWR
- J5 pad 2: Net-(J5-Pin_2) -> GNDS
- J6 pad 1: SUPP_PWR -> Net-(J6-Pin_1)
- J7 pad 1: Net-(J7-Pin_1) -> FUSE_OUT
- J7 pad 2: GNDS -> Net-(J7-Pin_2)
- Q1 pad 1: SUPP_PWR -> Net-(J6-Pin_1)
- Q1 pad 2: DCDC_Gate -> Net-(J7-Pin_2)
- Q1 pad 3: (no net) -> GNDS
- Q1A2 pad 1: DCDC_Gate -> Supp_Gate
- Q1A2 pad 2: Net-(Q1A2-Pad2) -> Net-(Q1A1-Pad2)
- Q1A2 pad 3: Net-(F1-Pad1) -> Net-(F2-Pad1)
- Q1A3 pad 1: Supp_Gate -> DCDC_Gate
- Q1A3 pad 2: Net-(Q1A1-Pad2) -> Net-(Q1A3-Pad2)
- Q1A3 pad 3: Net-(F1-Pad1) -> DCDC_PWR
- Q1A4 pad 2: Net-(Q1A2-Pad2) -> Net-(Q1A3-Pad2)
- Q1A4 pad 3: DCDC_PWR -> Net-(F2-Pad1)
- Q2 pad 2: ZENER_GATE -> Supp_Drive
- Q2 pad 3: Supp_Gate -> DCDC_Gate
- Q2 pad 5: DCDC_Gate -> DCDC_Drive
- Q2 pad 6: DCDC_Gate -> Supp_Gate
- R2 pad 2: DCDC_Gate -> Supp_Gate
- R3 pad 1: ZENER_GATE -> DCDC_PWR
- R3 pad 2: GNDS -> Net-(DS2-A)
- R4 pad 1: DCDC_PWR -> SUPP_PWR
- R4 pad 2: Net-(DS2-A) -> DCDC_Gate
- TP2 pad 1: DCDC_PWR -> DCDC_Gate
- TP3 pad 1: ZENER_GATE -> DCDC_PWR
- TP4 pad 1: DCDC_Gate -> Supp_Gate
- TP5 pad 1: Supp_Gate -> GNDS
Routing:
- net SUPP_PWR: track 69.6 -> 112.5 mm
- net Supp_Gate: track 38.1 -> 75.5 mm
- net Net-(J1-Pin_1): track 0.00 -> 36.6 mm
- net Net-(J7-Pin_1): track 22.4 -> 0.00 mm
- net DCDC_Drive: track 0.00 -> 22.4 mm
- net DCDC_PWR: track 14.3 -> 34.5 mm, vias 2 -> 1
- net Supp_Drive: track 0.00 -> 19.3 mm
- net DCDC_Gate: track 47.4 -> 66.4 mm, vias 2 -> 1
- net ZENER_GATE: track 18.2 -> 0.00 mm
- net Net-(Q1A2-Pad2): track 12.4 -> 0.00 mm
- net Net-(Q1A3-Pad2): track 0.00 -> 11.4 mm
- net Net-(J6-Pin_1): track 0.00 -> 8.76 mm
- net Net-(U1-A2): track 0.00 -> 6.96 mm
- net Net-(F2-Pad1): track 0.00 -> 3.40 mm
- net GNDS: vias 23 -> 19
- added copper zone on F.Cu, net DCDC_PWR
- added copper zone on B.Cu, net Net-(F2-Pad1)
- added copper zone on B.Cu, net Net-(J1-Pin_1)
- added copper zone on F.Cu, net Net-(J7-Pin_2)
- removed copper zone on B.Cu, net DCDC_PWR
- removed copper zone on B.Cu, net Net-(F1-Pad1)
- removed copper zone on F.Cu, net Net-(J5-Pin_2)
- removed copper zone on F.Cu, net SUPP_PWR

Commit message: silkscreen changes
Parts:
- LOGO2: moved to B.Cu
- moved LOGO2 226.4 mm to (130.5, 65.1), turned to 180 degrees
- moved LOGO1 147.1 mm to (53.3, 34.1)
- moved DS1 5.01 mm to (132.6, 52.4)
- moved R1 5.01 mm to (128.8, 52.4)
- moved TP5 5.00 mm to (138.0, 48.0)
Routing:
- net SUPP_PWR: track 112.5 -> 118.8 mm
- net Net-(F2-Pad1): track 3.40 -> 0.00 mm
- net GNDS: vias 19 -> 28

Commit message: changes
Parts:
- moved Q1A3 1.73 mm to (110.8, 56.5)
- moved Q1A4 1.10 mm to (110.8, 62.8)
- moved Q1A2 0.44 mm to (110.8, 69.1)
Routing:
- net Net-(J1-Pin_1): track 36.6 -> 0.00 mm
- net DCDC_PWR: track 34.5 -> 27.7 mm
- net DCDC_Gate: track 66.4 -> 72.6 mm
- net Net-(Q1A3-Pad2): track 11.4 -> 12.6 mm
- net Net-(Q1A1-Pad2): track 11.4 -> 12.3 mm
- net SUPP_PWR: track 118.8 -> 119.4 mm
Changed lines of the file:
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@@
 	(footprint "UTSVT_PowerSupp:SUP90P06-PCHAN-ENH-PWR-MOSFET"
 		(layer "F.Cu")
-		(at 110.8 69.5425)
+		(at 110.77 69.1)
 		(descr "TO-220AB-ren1")
 		(tags "Transistor")
@@
 	(footprint "UTSVT_PowerSupp:SUP90P06-PCHAN-ENH-PWR-MOSFET"
 		(layer "F.Cu")
-		(at 110.8325 63.9)
+		(at 110.82 62.8)
 		(descr "TO-220AB-ren1")
 		(tags "Transistor")
@@
 	(footprint "UTSVT_PowerSupp:SUP90P06-PCHAN-ENH-PWR-MOSFET"
 		(layer "F.Cu")
-		(at 110.8325 58.225)
+		(at 110.8325 56.5)
 		(descr "TO-220AB-ren1")
 		(tags "Transistor")
@@
 	)
 	(via
-		(at 108.4 97.4)
+		(at 110.4 97.3)
 		(size 0.8)
 		(drill 0.4)
@@
 	)
 	(segment
-		(start 117.7 73.4375)
-		(end 115.88 75.2575)
-		(width 0.25)
+		(start 113.4585 84.0385)
+		(end 110.9 81.48)
+		(width 0.5)
 		(layer "F.Cu")
 		(net 6)
 	)
 	(segment
-		(start 112.8 97.3)
-		(end 112.8 83.38)
-		(width 0.5)
+		(start 117.7 73.4375)
+		(end 115.88 75.2575)
+		(width 0.25)
 		(layer "F.Cu")
 		(net 6)
@@
 	)
 	(segment
+		(start 112.8 97.3)
+		(end 113.4585 96.6415)
+		(width 0.5)
+		(layer "F.Cu")
+		(net 6)
+	)
+	(segment
 		(start 111.7 98.4)
 		(end 112.8 97.3)
@@
 	)
 	(segment
+		(start 113.4585 96.6415)
+		(end 113.4585 84.0385)
+		(width 0.5)
+		(layer "F.Cu")
+		(net 6)
+	)
+	(segment
 		(start 114.2682 66.1)
 		(end 114.2682 66.1)
@@
 	)
 	(segment
-		(start 112.8 83.38)
-		(end 110.9 81.48)
-		(width 0.5)
-		(layer "F.Cu")
-		(net 6)
-	)
-	(segment
 		(start 106.1125 56.097436)
 		(end 116.009936 46.2)
@@
 	)
 	(segment
-		(start 124.7 63.4)
-		(end 126.68 65.38)
-		(width 0.25)
-		(layer "F.Cu")
-		(net 7)
-	)
-	(segment
 		(start 143 48)
 		(end 143 48.4)
@@
 	)
 	(segment
-		(start 143 48.4)
-		(end 151 56.4)
-		(width 0.25)
-		(layer "F.Cu")
-		(net 7)
-	)
-	(segment
-		(start 115.9125 58.225)
-		(end 116.825 58.225)
-		(width 0.25)
-		(layer "F.Cu")
-		(net 7)
-	)
-	(segment
-		(start 126.68 65.38)
-		(end 126.68 74.2875)
+		(start 126.68 74.2875)
+		(end 126.68 58.42)
 		(width 0.25)
 		(layer "F.Cu")
@@
 	)
 	(segment
-		(start 116.825 58.225)
-		(end 122 63.4)
-		(width 0.25)
-		(layer "F.Cu")
-		(net 7)
-	)
-	(segment
-		(start 122 63.4)
-		(end 124.7 63.4)
+		(start 143 48.4)
+		(end 151 56.4)
 		(width 0.25)
 		(layer "F.Cu")
@@
 	)
 	(segment
-		(start 110.8 69.5425)
-		(end 109.2575 69.5425)
+		(start 110.8 75.2575)
+		(end 110.8 69.13)
 		(width 0.5)
 		(layer "F.Cu")
@@
 	)
 	(segment
-		(start 110.8 75.2575)
-		(end 110.8 69.5425)
+		(start 115.9 45.6)
+		(end 120.8 45.6)
 		(width 0.5)
 		(layer "F.Cu")
@@
 	)
 	(segment
-		(start 104.6 56.9)
-		(end 115.9 45.6)
+		(start 110.77 69.1)
+		(end 110.75 69.1)
 		(width 0.5)
 		(layer "F.Cu")
@@
 	)
 	(segment
-		(start 114.8125 99.125)
-		(end 114.8375 99.15)
+		(start 120.8 45.6)
+		(end 123.2 48)
 		(width 0.5)
 		(layer "F.Cu")
@@
 	)
 	(segment
-		(start 115.9 45.6)
-		(end 120.8 45.6)
+		(start 110.8 69.13)
+		(end 110.77 69.1)
+		(width 0.5)
+		(layer "F.Cu")
+		(net 8)
+	)
+	(segment
+		(start 114.8125 99.125)
+		(end 114.8375 99.15)
 		(width 0.5)
 		(layer "F.Cu")
@@
 	)
 	(segment
-		(start 120.8 45.6)
-		(end 123.2 48)
+		(start 104.6 64.509936)
+		(end 104.6 56.9)
 		(width 0.5)
 		(layer "F.Cu")
@@
 	)
 	(segment
-		(start 104.6 64.885)
-		(end 104.6 56.9)
+		(start 104.6 56.9)
+		(end 115.9 45.6)
 		(width 0.5)
 		(layer "F.Cu")
@@
 	)
 	(segment
+		(start 110.75 69.1)
+		(end 108.252 66.602)
+		(width 0.5)
+		(layer "F.Cu")
+		(net 8)
+	)
+	(segment
 		(start 112.8 99.125)
 		(end 114.0855 97.8395)
@@
 	)
 	(segment
-		(start 109.2575 69.5425)
-		(end 104.6 64.885)
+		(start 106.692064 66.602)
+		(end 104.6 64.509936)
+		(width 0.5)
+		(layer "F.Cu")
+		(net 8)
+	)
+	(segment
+		(start 108.252 66.602)
+		(end 106.692064 66.602)
 		(width 0.5)
 		(layer "F.Cu")
@@
 	)
 	(segment
+		(start 110.8325 55.4555)
+		(end 110.8325 62.7)
+		(width 0.5)
+		(layer "F.Cu")
+		(net 9)
+	)
+	(segment
 		(start 117.0375 97.85)
 		(end 119.05 97.85)
@@
 	)
 	(segment
-		(start 110.8325 63.9)
-		(end 110.8325 58.225)
-		(width 0.5)
-		(layer "F.Cu")
-		(net 9)
-	)
-	(segment
-		(start 110.8325 58.225)
+		(start 118.288 48)
 		(end 110.8325 55.4555)
 		(width 0.5)
@@
 	)
 	(segment
-		(start 110.8325 55.4555)
-		(end 118.288 48)
+		(start 109.6325 63.9)
+		(end 106.2 63.9)
 		(width 0.5)
 		(layer "F.Cu")
@@
 	)
 	(segment
-		(start 110.8325 63.9)
-		(end 106.2 63.9)
+		(start 110.8325 62.7)
+		(end 109.6325 63.9)
 		(width 0.5)
 		(layer "F.Cu")
@@
 	)
 	(segment
-		(start 105.733 83.734084)
-		(end 117.0625 95.063584)
+		(start 110.8325 62.7)
+		(end 110.82 62.7125)
 		(width 0.5)
 		(layer "B.Cu")
@@
 	)
 	(segment
-		(start 105.733 68.9995)
-		(end 105.733 83.734084)
+		(start 104 84.1)
+		(end 105.1 85.2)
 		(width 0.5)
 		(layer "B.Cu")
@@
 	)
 	(segment
-		(start 117.0625 95.063584)
+		(start 117.0625 89.889212)
 		(end 117.0625 97.772998)
 		(width 0.5)
@@
 	)
 	(segment
-		(start 110.8325 63.9)
-		(end 105.733 68.9995)
+		(start 112.373288 85.2)
+		(end 117.0625 89.889212)
 		(width 0.5)
 		(layer "B.Cu")
@@
 	)
 	(segment
-		(start 113.34 69.5425)
-		(end 113.34 75.2575)
-		(width 2.5)
-		(layer "F.Cu")
-		(net 10)
+		(start 104 70.7325)
+		(end 104 84.1)
+		(width 0.5)
+		(layer "B.Cu")
+		(net 9)
 	)
 	(segment
-		(start 113.34 69.5425)
-		(end 113.34 75.2575)
-		(width 2.5)
+		(start 110.82 63.9125)
+		(end 104 70.7325)
+		(width 0.5)
 		(layer "B.Cu")
-		(net 10)
+		(net 9)
 	)
 	(segment
-		(start 104.5 63.5)
-		(end 100.5 67.5)
-		(width 4)
+		(start 110.82 62.7125)
+		(end 110.82 63.9125)
+		(width 0.5)
 		(layer "B.Cu")
-		(net 12)
+		(net 9)
 	)
 	(segment
-		(start 99.58 96.48)
-		(end 99.58 91.55)
-		(width 4)
+		(start 105.1 85.2)
+		(end 112.373288 85.2)
+		(width 0.5)
 		(layer "B.Cu")
-		(net 12)
+		(net 9)
 	)
 	(segment
-		(start 105.3 102.2)
-		(end 99.58 96.48)
-		(width 4)
-		(layer "B.Cu")
-		(net 12)
+		(start 113.34 69.13)
+		(end 113.34 75.2575)
+		(width 2.5)
+		(layer "F.Cu")
+		(net 10)
 	)
 	(segment
-		(start 104.5 49.5)
-		(end 104.5 63.5)
-		(width 4)
-		(layer "B.Cu")
-		(net 12)
+		(start 113.31 69.1)
+		(end 113.34 69.13)
+		(width 2.5)
+		(layer "F.Cu")
+		(net 10)
 	)
 	(segment
-		(start 105.3 104)
-		(end 105.3 102.2)
-		(width 4)
+		(start 113.31 69.1)
+		(end 113.34 69.13)
+		(width 2.5)
 		(layer "B.Cu")
-		(net 12)
+		(net 10)
 	)
 	(segment
-		(start 106 48)
-		(end 104.5 49.5)
-		(width 4)
+		(start 113.34 69.13)
+		(end 113.34 75.2575)
+		(width 2.5)
 		(layer "B.Cu")
-		(net 12)
+		(net 10)
 	)
 	(segment
@@
 	)
 	(segment
-		(start 113.3725 58.225)
-		(end 113.3725 63.9)
+		(start 113.3725 56.5)
+		(end 113.3725 62.7875)
 		(width 2.5)
 		(layer "F.Cu")
@@
 	)
 	(segment
-		(start 113.3675 58.1675)
-		(end 113.3675 63.8825)
+		(start 113.3725 62.7875)
+		(end 113.36 62.8)
+		(width 2.5)
+		(layer "F.Cu")
+		(net 16)
+	)
+	(segment
+		(start 113.3675 56.505)
+		(end 113.3675 62.7925)
+		(width 2.5)
+		(layer "B.Cu")
+		(net 16)
+	)
+	(segment
+		(start 113.3725 56.5)
+		(end 113.3675 56.505)
+		(width 2.5)
+		(layer "B.Cu")
+		(net 16)
+	)
+	(segment
+		(start 113.3675 62.7925)
+		(end 113.36 62.8)
 		(width 2.5)
 		(layer "B.Cu")
@@
 		(polygon
 			(pts
-				(xy 94.2 65.3) (xy 103.4 65.3) (xy 103.4 88.1) (xy 114 88.1) (xy 114 94.4) (xy 94.2 94.4) (xy 94.2 93.7)
+				(xy 103.5 94.4) (xy 103.5 106.3) (xy 109.4 106.3) (xy 109.4 94.4) (xy 113.8 94.4) (xy 113.8 88.1)
+				(xy 103.2 88.1) (xy 103.1 88) (xy 103.1 50) (xy 107.6 50) (xy 107.6 45.9) (xy 94.5 45.9) (xy 94.5 94.4)
 			)
 		)

Commit message: changes
Parts:
- added DS3: DCDC_PWR, Diode_SMD:D_0805_2012Metric, F.Cu at (117.8, 82.8)
- added DS4: DCDC_PWR, Diode_SMD:D_0805_2012Metric, F.Cu at (117.9, 87.2)
- added R10: 5.1K, Resistor_SMD:R_0805_2012Metric, F.Cu at (115.7, 87.2)
- added R9: 5.1K, Resistor_SMD:R_0805_2012Metric, F.Cu at (115.8, 82.8)
Routing:
- net SUPP_PWR: track 119.4 -> 113.4 mm
- net DCDC_Drive: track 22.4 -> 27.1 mm
- net Supp_Drive: track 19.3 -> 23.4 mm
- net Net-(DS4-A): track 0.00 -> 2.17 mm
- net Net-(DS3-A): track 0.00 -> 2.11 mm
- net GNDS: track 0.00 -> 0.76 mm
- net DCDC_Gate: track 72.6 -> 72.7 mm, vias 1 -> 3

Commit message: changes
Routing:
- net Supp_Drive: track 23.4 -> 23.9 mm, vias 0 -> 1
Changed lines of the file:
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@@
 	)
 	(segment
-		(start 117.5305 84.477)
-		(end 121.283 84.477)
+		(start 115.7075 86.3)
+		(end 114.356 87.6515)
+		(width 0.25)
+		(layer "F.Cu")
+		(net 17)
+	)
+	(segment
+		(start 115.75 86.2575)
+		(end 115.75 86.3)
 		(width 0.25)
 		(layer "F.Cu")
@@
 	(segment
 		(start 115.735 86.2725)
-		(end 114.356 87.6515)
-		(width 0.25)
-		(layer "F.Cu")
-		(net 17)
-	)
-	(segment
-		(start 121.283 84.477)
-		(end 123.26 82.5)
+		(end 115.75 86.2575)
 		(width 0.25)
 		(layer "F.Cu")
@@
 	)
 	(segment
+		(start 115.75 86.3)
+		(end 115.7075 86.3)
+		(width 0.25)
+		(layer "F.Cu")
+		(net 17)
+	)
+	(segment
 		(start 116.127 98.2145)
 		(end 116.4125 98.5)
@@
 		(net 17)
 	)
-	(segment
-		(start 115.735 86.2725)
-		(end 117.5305 84.477)
-		(width 0.25)
-		(layer "F.Cu")
+	(via
+		(at 115.75 86.3)
+		(size 0.8)
+		(drill 0.4)
+		(layers "F.Cu" "B.Cu")
 		(net 17)
 	)
+	(segment
+		(start 118.75 82.5)
+		(end 123.26 82.5)
+		(width 0.25)
+		(layer "B.Cu")
+		(net 17)
+	)
+	(segment
+		(start 115.75 85.5)
+		(end 118.75 82.5)
+		(width 0.25)
+		(layer "B.Cu")
+		(net 17)
+	)
+	(segment
+		(start 115.75 86.3)
+		(end 115.75 85.5)
+		(width 0.25)
+		(layer "B.Cu")
+		(net 17)
+	)

Commit message: PCB changes
Parts:
- moved Q2 24.4 mm to (117.6, 74.2)
- moved R4 19.0 mm to (103.6, 81.8), turned to 90 degrees
- moved R7 17.5 mm to (114.8, 80.8), turned to 0 degrees
- moved R8 16.2 mm to (114.8, 83.0), turned to 0 degrees
- moved DS1 13.0 mm to (121.2, 46.2), turned to -90 degrees
- moved DS4 12.0 mm to (120.0, 99.0)
- moved R10 12.0 mm to (117.8, 99.0)
- moved DS3 10.6 mm to (119.9, 93.2)
- moved R9 10.6 mm to (117.8, 93.3)
- moved TP1 10.0 mm to (118.1, 48.0)
- moved TP4 9.83 mm to (133.0, 48.0)
- moved TP2 9.71 mm to (128.0, 48.0)
- moved R2 9.09 mm to (107.7, 81.8), turned to 90 degrees
- moved U1 8.55 mm to (130.9, 86.0)
- moved R1 7.99 mm to (121.2, 50.0), turned to 90 degrees
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Routing:
- net SUPP_PWR: track 113.4 -> 70.6 mm, vias 0 -> 2
- net DCDC_Gate: track 72.7 -> 84.4 mm, vias 3 -> 2
- net Supp_Gate: track 75.7 -> 83.2 mm, vias 0 -> 6
- net Net-(Q1A3-Pad2): track 12.6 -> 7.00 mm
- net DCDC_PWR: track 27.7 -> 22.2 mm
- net Net-(Q1A1-Pad2): track 12.3 -> 7.00 mm
- net Supp_Drive: track 23.9 -> 29.0 mm, vias 1 -> 0
- net DCDC_Drive: track 27.1 -> 24.0 mm, vias 0 -> 2
- net GNDS: track 0.76 -> 1.36 mm, vias 28 -> 31
- net Net-(J6-Pin_1): track 8.76 -> 8.16 mm
- added copper zone on F.Cu, net SUPP_PWR
- removed copper zone on B.Cu, net SUPP_PWR
Other:
- board size 82 x 66 mm -> 87 x 71 mm

Commit message: pcb changes
Parts:
- removed R2, R4: 100k, Resistor_SMD:R_0805_2012Metric
- moved R6 2.40 mm to (127.0, 80.2)
Routing:
- net Net-(Q1A1-Pad2): track 7.00 -> 14.0 mm
- net Net-(Q1A3-Pad2): track 7.00 -> 13.9 mm
- net Supp_Gate: track 83.2 -> 81.0 mm
- net Net-(U1-A2): track 7.33 -> 8.58 mm
- net DCDC_Gate: track 84.4 -> 83.5 mm, vias 2 -> 4
- net GNDS: vias 31 -> 27
- net FUSE_OUT: vias 0 -> 3
- added copper zone on F.Cu, net FUSE_OUT
- added copper zone on F.Cu, net Net-(F2-Pad1)
- added copper zone on F.Cu, net Net-(J1-Pin_1)
- removed copper zone on B.Cu, net FUSE_OUT
- removed copper zone on B.Cu, net Net-(F2-Pad1)
- removed copper zone on B.Cu, net Net-(J1-Pin_1)
