File: Power-Secondary.kicad_pcb (KiCad board)
At the start: 2 copper layers, 87 x 71 mm, 44 parts, among them J1 SUPP PWR 1, J2 SUPP PWR 2, J3 SUPP OUT, J4 SUPP PWR MON, J5 DCDC SUPPLY, J6 LV ENABLE, J7 FUSE OUT, Q1 FDD86250-F085, Q1A1 IRFU5305PbF, Q1A2 IRFU5305PbF, Q1A3 IRFU5305PbF, Q1A4 IRFU5305PbF, Q2 S1G1D2S2G2D1, U1 Nucleo_L432KC

Commit message: Schematic redesign
Parts:
- removed DS3, DS4: DCDC_PWR, Diode_SMD:D_0805_2012Metric
- removed TP1: SUPP_PWR, TestPoint:TestPoint_Pad_2.0x2.0mm
- removed TP2: DCDC_Gate, TestPoint:TestPoint_Pad_2.0x2.0mm
- removed TP3: DCDC_PWR, TestPoint:TestPoint_Pad_2.0x2.0mm
- removed TP4: Supp_Gate, TestPoint:TestPoint_Pad_2.0x2.0mm
- added C5: 100uF, Capacitor_SMD:C_1210_3225Metric, B.Cu at (200.0, 40.0)
- added C6: 100uF, Capacitor_SMD:C_1210_3225Metric, B.Cu at (200.0, 44.2)
- added C7: 100uF, Capacitor_SMD:C_1210_3225Metric, B.Cu at (200.0, 48.5)
- added DCDC_PWR1: DCDC_PWR, TestPoint:TestPoint_Pad_2.0x2.0mm, F.Cu at (168.0, 26.5)
- added D_GATE1: DCDC_Gate, TestPoint:TestPoint_Pad_2.0x2.0mm, F.Cu at (174.5, 26.5)
- added F3: Fuse, Fuse:Fuseholder_Blade_Mini_Keystone_3568, F.Cu at (171.0, 42.0)
- added F4: Fuse, Fuse:Fuseholder_Blade_Mini_Keystone_3568, F.Cu at (190.8, 58.0)
- added GND1: GND, TestPoint:TestPoint_Pad_2.0x2.0mm, F.Cu at (161.5, 36.0)
- added J8: Fan OUT, Connector_Molex:Molex_Sabre_43160-0102_1x02_P7.49mm_Vertical, F.Cu at (197.0, 33.8)
- added Q1A5: IRFU5305PbF, UTSVT_PowerSupp:SUP90P06-PCHAN-ENH-PWR-MOSFET, F.Cu at (173.5, 52.3)
- added Q1A6: IRFU5305PbF, UTSVT_PowerSupp:SUP90P06-PCHAN-ENH-PWR-MOSFET, F.Cu at (206.5, 50.6)
- added Q1A7: IRFU5305PbF, UTSVT_PowerSupp:SUP90P06-PCHAN-ENH-PWR-MOSFET, F.Cu at (173.5, 60.1)
- added Q1A8: IRFU5305PbF, UTSVT_PowerSupp:SUP90P06-PCHAN-ENH-PWR-MOSFET, F.Cu at (211.5, 58.4)
- added Q3: S1G1D2S2G2D1, UTSVT_PowerSupp:SOT65P210X100-6N, F.Cu at (177.0, 100.5)
- added Q4: FDD86250-F085, UTSVT_PowerSupp:FDD13AN06A0F085, B.Cu at (208.1, 42.7)
- added SUPP_PWR1: SUPP_PWR, TestPoint:TestPoint_Pad_2.0x2.0mm, F.Cu at (168.0, 31.0)
- added TP7: Supp_Gate2, TestPoint:TestPoint_Pad_2.0x2.0mm, F.Cu at (161.5, 31.0)
- C4, LOGO1, Q1, R8: moved to B.Cu
- R10: value 5.1K -> 100k; moved to B.Cu
- R5, R6: moved to F.Cu
- R9: value 5.1K -> 100k
- TP5: value GND -> Supp_Gate
- TP6: value GND -> DCDC_Gate2
- moved LOGO1 174.3 mm to (213.0, 104.0), turned to 180 degrees
- moved H3 128.3 mm to (216.0, 117.5)
- moved Q1A4 106.0 mm to (211.5, 67.0), turned to 180 degrees
- moved Q1A3 103.0 mm to (206.5, 76.0)
- moved R8 90.5 mm to (200.0, 52.5)
- moved J6 86.8 mm to (182.0, 27.1), turned to 0 degrees
- moved R10 85.7 mm to (200.0, 74.5), turned to 0 degrees
- moved C4 82.1 mm to (201.5, 116.5), turned to 180 degrees
- moved R5 80.6 mm to (205.0, 94.4)
- moved R6 80.1 mm to (205.0, 98.4)
- moved J4 77.9 mm to (155.5, 108.5), turned to 90 degrees
- moved F1 69.8 mm to (171.0, 80.5), turned to 0 degrees
- moved H1 69.8 mm to (155.0, 28.5)
- moved Q1A2 68.0 mm to (173.5, 67.6)
- moved Q1A1 68.0 mm to (173.5, 74.8)
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Connections:
- net Net-(F2-Pad1) renamed OUT_1
- net Net-(J6-Pin_1) renamed LV_EN
- net Net-(J7-Pin_2) renamed DRAIN_1
- C4 pad 1: SUPP_PWR -> FUSE_OUT
- F1 pad 1: Net-(J1-Pin_1) -> SUPP_IN
- F1 pad 2: SUPP_PWR -> SUPP_PWR2
- J1 pad 1: Net-(J1-Pin_1) -> SUPP_IN
- J2 pad 1: Net-(J1-Pin_1) -> SUPP_IN
- J3 pad 1: Net-(J1-Pin_1) -> SUPP_IN
- J4 pad 1: Net-(J1-Pin_1) -> SUPP_IN
- Q1A1 pad 1: Supp_Gate -> Supp_Gate2
- Q1A1 pad 3: SUPP_PWR -> SUPP_PWR2
- Q1A2 pad 1: Supp_Gate -> Supp_Gate2
- Q1A3 pad 1: DCDC_Gate -> DCDC_Gate2
- Q1A4 pad 1: DCDC_Gate -> DCDC_Gate2
- Q2 pad 2: Supp_Drive -> /Nucleo-L432KC/Supp_Drive
- Q2 pad 3: DCDC_Gate -> Supp_Gate2
- Q2 pad 5: DCDC_Drive -> /Nucleo-L432KC/Supp_Drive2
- R10 pad 1: Supp_Drive -> SUPP_IN
- R10 pad 2: Net-(DS4-A) -> DCDC_Gate2
- R7 pad 1: SUPP_PWR -> SUPP_IN
- R8 pad 1: SUPP_PWR -> SUPP_IN
- R9 pad 1: DCDC_Drive -> SUPP_IN
- R9 pad 2: Net-(DS3-A) -> Supp_Gate2
- TP5 pad 1: GNDS -> Supp_Gate
- TP6 pad 1: GNDS -> DCDC_Gate2
- U1 pad 24: DCDC_Drive -> unconnected-(U1-A5-Pad24)
- U1 pad 25: Supp_Drive -> unconnected-(U1-A6-Pad25)
- U1 pad 30: SUPP_PWR -> FUSE_OUT
- U1 pad 6: unconnected-(U1-D3-Pad6) -> /Nucleo-L432KC/Supp_Drive2
- U1 pad 7: unconnected-(U1-D4-Pad7) -> /Nucleo-L432KC/DCDC_Drive2
- U1 pad 8: unconnected-(U1-D5-Pad8) -> /Nucleo-L432KC/Supp_Drive
- U1 pad 9: unconnected-(U1-D6-Pad9) -> /Nucleo-L432KC/DCDC_Drive
Routing:
- net DCDC_Gate2: track 0.00 -> 121.2 mm, vias 0 -> 2
- net LV_EN: track 8.16 -> 113.9 mm, vias 0 -> 2
- net SUPP_IN: track 0.00 -> 98.6 mm, vias 0 -> 2
- net Supp_Gate2: track 0.00 -> 86.9 mm, vias 0 -> 2
- net SUPP_PWR: track 70.6 -> 21.2 mm, vias 2 -> 0
- net DCDC_Gate: track 83.5 -> 126.0 mm, vias 4 -> 2
- net DCDC_PWR: track 22.5 -> 60.6 mm
- net FUSE_OUT: track 0.00 -> 35.8 mm, vias 3 -> 1
- net Net-(Q1A5-Pad2): track 0.00 -> 31.0 mm
- net Net-(U1-A2): track 8.58 -> 37.9 mm, vias 0 -> 1
- net Supp_Drive: track 29.0 -> 0.00 mm
- net DCDC_Drive: track 24.0 -> 0.00 mm, vias 2 -> 0
- net Net-(Q1A6-Pad2): track 0.00 -> 23.5 mm
- net /Nucleo-L432KC/Supp_Drive2: track 0.00 -> 23.5 mm, vias 0 -> 1
- net GNDS: track 1.36 -> 22.7 mm, vias 27 -> 7
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- added copper zone on F.Cu, net BPS/Fan OUT
- added copper zone on B.Cu, net DRAIN_1
- added copper zone on B.Cu, net DRAIN_2
- added copper zone on F.Cu, net OUT_2
- added copper zone on F.Cu, net SUPP_IN
- added copper zone on F.Cu, net SUPP_PWR2
- removed copper zone on F.Cu, net DRAIN_1
- removed copper zone on F.Cu, net GNDS
- removed copper zone on F.Cu, net Net-(J1-Pin_1)
Other:
- board size 87 x 71 mm -> 71 x 99 mm
- copper layers 2 -> 4
- board text added: "DCDC_PWR"
- board text added: "D_GATE1"
- board text added: "D_GATE2"
- board text added: "Jason, Pratyush, Frank, Jack Board"
- board text added: "SGATE_1"
- board text added: "SGATE_2"
- board text added: "SUPP_PWR"
- board text removed: "DCDC GATE"
- board text removed: "DCDC PWR"
- board text removed: "FUSE OUT"
- board text removed: "Jason and Pratyush"
- board text removed: "LV ENABLE"
- board text removed: "SUPP GATE"
- board text removed: "SUPP MON"
- board text removed: "SUPP OUT"
- board text removed: "SUPP PWR"
- board text removed: "SUPP PWR 1"
- board text removed: "SUPP PWR 2"
- board text removed: "ZENER GATE"
- board text removed: "{dblquote}Rabid{dblquote}, not rabbit."
