File: _autosave-switch.kicad_sch (KiCad schematic)
At the start: 10 parts, among them J9 OUT, Q1A10 IRFU5305PbF, Q1A11 IRFU5305PbF, Q1A12 IRFU5305PbF, Q1A9 IRFU5305PbF, Q5 FDD86250-F085

Commit message: layout changes
Connections:
- net Fuse_Out: now reaches C10.1, C8.1, C9.1, F5.2, J9.1 (Pin_1)
Changed lines of the file:
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@@
+		)
+	)
+	(hierarchical_label "Fuse_Out"
+		(shape output)
+		(at 161.036 108.204 90)
+		(fields_autoplaced yes)
+		(effects
+			(font
+				(size 1.27 1.27)
+			)
+			(justify left)
 		)
 	)
