File: nmos.kicad_sch (KiCad schematic)
At the start: 6 parts, among them Q2 S1G1D2S2G2D1, Q5 S1G1D2S2G2D1

Commit message: Schematic redesign
Parts:
- removed Q5: S1G1D2S2G2D1, UTSVT_PowerSupp:SOT65P210X100-6N, symbol Device:Q_Dual_NMOS_S1G1D2S2G2D1
- added Q3: S1G1D2S2G2D1, UTSVT_PowerSupp:SOT65P210X100-6N, symbol Device:Q_Dual_NMOS_S1G1D2S2G2D1
Connections:
- net DCDC_Drive: now also Q3.2 (G); no longer Q2.5 (G)
- net DCDC_Drive2: now also Q3.5 (G)
- net DCDC_Gate: now also Q3.6 (D); no longer Q2.3 (D)
- net DCDC_Gate2: now also Q3.3 (D)
- net GNDS: now also Q3.1 (S), Q3.4 (S)
- net Supp_Drive2: now also Q2.5 (G)
- net Supp_Gate2: now also Q2.3 (D)

Commit message: sch changes
Connections:
- net DCDC_Drive: now also Q2.5 (G); no longer Q3.2 (G)
- net DCDC_Gate: now also Q2.3 (D), R9.2; no longer Q3.6 (D), R8.2
- net Supp_Drive2: now also Q3.2 (G); no longer Q2.5 (G)
- net Supp_Gate2: now also Q3.6 (D), R8.2; no longer Q2.3 (D), R9.2
Changed lines of the file:
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@@
+	)
+	(junction
+		(at 177.8 106.172)
+		(diameter 0)
+		(color 0 0 0 0)
 	)
 	(junction
@@
 	)
 	(junction
-		(at 177.8 106.045)
-		(diameter 0)
-		(color 0 0 0 0)
-	)
-	(junction
 		(at 177.8 76.2)
 		(diameter 0)
@@
 	(wire
 		(pts
-			(xy 177.8 104.775) (xy 177.8 106.045)
+			(xy 177.8 106.172) (xy 177.8 107.315)
 		)
 		(stroke
@@
 	(wire
 		(pts
+			(xy 120.396 110.49) (xy 121.285 110.49)
+		)
+		(stroke
+			(width 0)
+			(type default)
+		)
+	)
+	(wire
+		(pts
 			(xy 227.33 106.68) (xy 222.25 106.68)
 		)
@@
 	(wire
 		(pts
+			(xy 128.905 104.14) (xy 134.112 104.14)
+		)
+		(stroke
+			(width 0)
+			(type default)
+		)
+	)
+	(wire
+		(pts
 			(xy 78.74 104.14) (xy 78.74 105.41)
 		)
@@
 	(wire
 		(pts
+			(xy 177.8 104.775) (xy 177.8 106.172)
+		)
+		(stroke
+			(width 0)
+			(type default)
+		)
+	)
+	(wire
+		(pts
 			(xy 78.74 104.14) (xy 83.82 104.14)
 		)
@@
 	(wire
 		(pts
+			(xy 170.18 112.522) (xy 170.18 112.395)
+		)
+		(stroke
+			(width 0)
+			(type default)
+		)
+	)
+	(wire
+		(pts
 			(xy 78.74 76.2) (xy 78.74 95.25)
 		)
@@
 	(wire
 		(pts
-			(xy 177.8 106.045) (xy 177.8 107.315)
-		)
-		(stroke
-			(width 0)
-			(type default)
-		)
-	)
-	(wire
-		(pts
 			(xy 177.8 76.2) (xy 177.8 97.155)
 		)
@@
 	(wire
 		(pts
-			(xy 128.905 104.14) (xy 133.985 104.14)
+			(xy 168.91 112.522) (xy 170.18 112.522)
 		)
 		(stroke
@@
 	(wire
 		(pts
-			(xy 182.88 106.045) (xy 177.8 106.045)
+			(xy 182.88 106.172) (xy 177.8 106.172)
 		)
 		(stroke
@@
 	(hierarchical_label "DCDC_Drive"
 		(shape input)
-		(at 170.18 112.395 180)
+		(at 120.396 110.49 180)
 		(fields_autoplaced yes)
 		(effects
@@
 	(hierarchical_label "DCDC_Gate"
 		(shape output)
-		(at 182.88 106.045 0)
+		(at 134.112 104.14 0)
 		(fields_autoplaced yes)
 		(effects
@@
 	(hierarchical_label "Supp_Gate2"
 		(shape output)
-		(at 133.985 104.14 0)
+		(at 182.88 106.172 0)
 		(fields_autoplaced yes)
 		(effects
@@
 	(hierarchical_label "Supp_Drive2"
 		(shape input)
-		(at 121.285 110.49 180)
-		(fields_autoplaced yes)
-		(effects
+		(at 168.91 112.522 180)
+		(fields_autoplaced yes)
+		(effects

Commit message: layout changes
Connections:
- net DCDC_Drive renamed FUSEOUT_DCDC_Drive
- net DCDC_Drive2 renamed BPS_DCDC_Drive
- net DCDC_Gate renamed FUSEOUT_DCDC_Gate
- net DCDC_Gate2 renamed BPS_DCDC_Gate
- net Supp_Drive renamed FUSEOUT_Supp_Drive
- net Supp_Drive2 renamed BPS_Supp_Drive
- net Supp_Gate renamed FUSEOUT_Supp_Gate
- net Supp_Gate2 renamed BPS_Supp_Gate
Changed lines of the file:
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@@
 		)
 	)
-	(hierarchical_label "DCDC_Drive"
+	(hierarchical_label "FUSEOUT_DCDC_Drive"
 		(shape input)
 		(at 120.396 110.49 180)
@@
 		)
 	)
-	(hierarchical_label "Supp_Drive"
+	(hierarchical_label "FUSEOUT_Supp_Drive"
 		(shape input)
 		(at 71.12 110.49 180)
@@
 		)
 	)
-	(hierarchical_label "Supp_Gate"
+	(hierarchical_label "FUSEOUT_Supp_Gate"
 		(shape output)
 		(at 83.82 104.14 0)
@@
 		)
 	)
-	(hierarchical_label "DCDC_Gate2"
+	(hierarchical_label "BPS_DCDC_Gate"
 		(shape output)
 		(at 227.33 106.68 0)
@@
 		)
 	)
-	(hierarchical_label "DCDC_Gate"
+	(hierarchical_label "FUSEOUT_DCDC_Gate"
 		(shape output)
 		(at 134.112 104.14 0)
@@
 		)
 	)
-	(hierarchical_label "Supp_Gate2"
+	(hierarchical_label "BPS_Supp_Gate"
 		(shape output)
 		(at 182.88 106.172 0)
@@
 		)
 	)
-	(hierarchical_label "Supp_Drive2"
+	(hierarchical_label "BPS_Supp_Drive"
 		(shape input)
 		(at 168.91 112.522 180)
@@
 		)
 	)
-	(hierarchical_label "DCDC_Drive2"
+	(hierarchical_label "BPS_DCDC_Drive"
 		(shape input)
 		(at 214.63 113.03 180)
