File: testpoints.kicad_sch (KiCad schematic)
At the start: 11 parts

Commit message: Schematic redesign
Parts:
- renumbered TP2 to DCDC_PWR1, TP4 to D_GATE1, TP3 to GND1, TP1 to SUPP_PWR1
Changed lines of the file:
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@@
 		(on_board yes)
 		(dnp no)
-		(property "Reference" "TP3"
+		(property "Reference" "GND1"
 			(at 183.8452 87.376 0)
 			(effects
@@
 			(project "Power-Secondary"
 				(path "/ba21eba1-72a9-489c-9498-a38516b9f252/3e7100ec-df3a-4713-932e-67c755937c6c"
-					(reference "TP3")
+					(reference "GND1")
 					(unit 1)
 				)
@@
 		(on_board yes)
 		(dnp no)
-		(property "Reference" "TP4"
+		(property "Reference" "D_GATE1"
 			(at 141.4272 108.204 0)
 			(effects
@@
 			(project "Power-Secondary"
 				(path "/ba21eba1-72a9-489c-9498-a38516b9f252/3e7100ec-df3a-4713-932e-67c755937c6c"
-					(reference "TP4")
+					(reference "D_GATE1")
 					(unit 1)
 				)
@@
 		(on_board yes)
 		(dnp no)
-		(property "Reference" "TP1"
+		(property "Reference" "SUPP_PWR1"
 			(at 139.3952 84.836 0)
 			(effects
@@
 			(project "Power-Secondary"
 				(path "/ba21eba1-72a9-489c-9498-a38516b9f252/3e7100ec-df3a-4713-932e-67c755937c6c"
-					(reference "TP1")
+					(reference "SUPP_PWR1")
 					(unit 1)
 				)
@@
 		(on_board yes)
 		(dnp no)
-		(property "Reference" "TP2"
+		(property "Reference" "DCDC_PWR1"
 			(at 163.5252 84.836 0)
 			(effects
@@
 			(project "Power-Secondary"
 				(path "/ba21eba1-72a9-489c-9498-a38516b9f252/3e7100ec-df3a-4713-932e-67c755937c6c"
-					(reference "TP2")
-					(unit 1)
-				)
+					(reference "DCDC_PWR1")
+					(unit 1)
+				)

Commit message: layout changes
Connections:
- net DCDC_Gate renamed FUSEOUT_DCDC_Gate
- net DCDC_Gate2 renamed BPS_DCDC_Gate
- net Supp_Gate renamed FUSEOUT_Supp_Gate
- net Supp_Gate2 renamed BPS_Supp_Gate
Other:
- moved on the sheet: TP5, TP7
Changed lines of the file:
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@@
 		)
 	)
-	(hierarchical_label "Supp_Gate"
+	(hierarchical_label "FUSEOUT_Supp_Gate"
 		(shape input)
-		(at 166.624 111.252 180)
+		(at 177.038 111.76 180)
 		(fields_autoplaced yes)
 		(effects
@@
 		)
 	)
-	(hierarchical_label "Supp_Gate2"
+	(hierarchical_label "BPS_Supp_Gate"
 		(shape input)
-		(at 166.878 120.65 180)
+		(at 177.292 121.158 180)
 		(fields_autoplaced yes)
 		(effects
@@
 		)
 	)
-	(hierarchical_label "DCDC_Gate"
+	(hierarchical_label "FUSEOUT_DCDC_Gate"
 		(shape input)
 		(at 139.954 111.252 180)
@@
 		)
 	)
-	(hierarchical_label "DCDC_Gate2"
+	(hierarchical_label "BPS_DCDC_Gate"
 		(shape input)
 		(at 140.208 120.65 180)
@@
 	(symbol
 		(lib_id "Connector:TestPoint")
-		(at 166.624 111.252 0)
+		(at 177.038 111.76 0)
 		(unit 1)
 		(exclude_from_sim no)
@@
 		(dnp no)
 		(property "Reference" "TP5"
-			(at 168.0972 108.204 0)
+			(at 178.5112 108.712 0)
 			(effects
 				(font
@@
 		)
 		(property "Value" "Supp_Gate"
-			(at 168.0972 110.5154 0)
+			(at 178.5112 111.0234 0)
 			(effects
 				(font
@@
 		)
 		(property "Footprint" "TestPoint:TestPoint_Pad_2.0x2.0mm"
-			(at 171.704 111.252 0)
+			(at 182.118 111.76 0)
 			(effects
 				(font
@@
 		)
 		(property "Datasheet" "~"
-			(at 171.704 111.252 0)
-			(effects
-				(font
-					(size 1.27 1.27)
-				)
-				(hide yes)
-			)
-		)
-		(property "Description" ""
-			(at 166.624 111.252 0)
+			(at 182.118 111.76 0)
+			(effects
+				(font
+					(size 1.27 1.27)
+				)
+				(hide yes)
+			)
+		)
+		(property "Description" ""
+			(at 177.038 111.76 0)
 			(effects
 				(font
@@
 		)
 		(property "Sim.Device" "SPICE"
-			(at 166.624 111.252 0)
+			(at 177.038 111.76 0)
 			(effects
 				(font
@@
 	(symbol
 		(lib_id "Connector:TestPoint")
-		(at 166.878 120.65 0)
+		(at 177.292 121.158 0)
 		(unit 1)
 		(exclude_from_sim no)
@@
 		(dnp no)
 		(property "Reference" "TP7"
-			(at 168.3512 117.602 0)
+			(at 178.7652 118.11 0)
 			(effects
 				(font
@@
 		)
 		(property "Value" "Supp_Gate2"
-			(at 168.3512 119.9134 0)
+			(at 178.7652 120.4214 0)
 			(effects
 				(font
@@
 		)
 		(property "Footprint" "TestPoint:TestPoint_Pad_2.0x2.0mm"
-			(at 171.958 120.65 0)
+			(at 182.372 121.158 0)
 			(effects
 				(font
@@
 		)
 		(property "Datasheet" "~"
-			(at 171.958 120.65 0)
-			(effects
-				(font
-					(size 1.27 1.27)
-				)
-				(hide yes)
-			)
-		)
-		(property "Description" ""
-			(at 166.878 120.65 0)
+			(at 182.372 121.158 0)
+			(effects
+				(font
+					(size 1.27 1.27)
+				)
+				(hide yes)
+			)
+		)
+		(property "Description" ""
+			(at 177.292 121.158 0)
 			(effects
 				(font
@@
 		)
 		(property "Sim.Device" "SPICE"
-			(at 166.878 120.65 0)
-			(effects
-				(font
+			(at 177.292 121.158 0)
+			(effects
+				(font
