File: LTC4421.kicad_sch (KiCad schematic)
At the start: 59 parts, among them U2 LTC4421CG-PBF, U3 74LVC2G07GV,125, U4 74LVC2G07GV,125, U5 74LVC2G07GV,125

Commit message: sch iteration 1 complete plssssssssss
Parts:
- renumbered CINTV_CC1 to CINTVCC1
Connections:
- net INTV_CC is gone; now on net INTVCC: CINTVCC1.1, U2.16 (CASIN), U2.17 (INTVCC)
Other:
- note added: "Notes: t_QUAL = C_QUAL * 16 (ms/nF) t_QUAL = 8 ms"
- note removed: "Notes: t_QUAL = C_QUAL * 16 (ms/nF) t_QUAL = 1 ms"
Changed lines of the file:
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@@
 	)
 	(junction
+		(at 29.21 68.58)
+		(diameter 0)
+		(color 0 0 0 0)
+	)
+	(junction
+		(at 31.75 66.04)
+		(diameter 0)
+		(color 0 0 0 0)
+	)
+	(junction
 		(at 223.52 73.66)
 		(diameter 0)
@@
 	(wire
 		(pts
+			(xy 29.21 68.58) (xy 31.75 68.58)
+		)
+		(stroke
+			(width 0)
+			(type default)
+		)
+	)
+	(wire
+		(pts
 			(xy 158.75 55.88) (xy 158.75 57.15)
 		)
@@
 	(wire
 		(pts
+			(xy 24.13 66.04) (xy 31.75 66.04)
+		)
+		(stroke
+			(width 0)
+			(type default)
+		)
+	)
+	(wire
+		(pts
 			(xy 270.51 148.59) (xy 270.51 160.02)
 		)
@@
 	(wire
 		(pts
-			(xy 24.13 68.58) (xy 31.75 68.58)
+			(xy 24.13 68.58) (xy 29.21 68.58)
 		)
 		(stroke
@@
 		)
 	)
-	(text "Notes:  \n  t_QUAL = C_QUAL * 16 (ms/nF)\n  t_QUAL = 1 ms"
+	(text "Notes:  \n  t_QUAL = C_QUAL * 16 (ms/nF)\n  t_QUAL = 8 ms"
 		(exclude_from_sim no)
 		(at 92.456 72.136 0)
@@
 		)
 	)
-	(label "INTV_CC"
+	(label "INTVCC"
 		(at 24.13 68.58 0)
 		(fields_autoplaced yes)
@@
 		)
 	)
-	(label "SHDN"
-		(at 77.47 66.04 180)
-		(fields_autoplaced yes)
-		(effects
-			(font
-				(size 1.27 1.27)
-			)
-			(justify right bottom)
-		)
-	)
 	(label "V2"
 		(at 90.17 173.99 0)
@@
 		)
 	)
-	(label "VALID2"
-		(at 77.47 60.96 180)
-		(fields_autoplaced yes)
-		(effects
-			(font
-				(size 1.27 1.27)
-			)
-			(justify right bottom)
-		)
-	)
 	(label "INTVCC"
 		(at 181.61 160.02 90)
@@
 		)
 	)
+	(hierarchical_label "VALID2"
+		(shape output)
+		(at 77.47 60.96 0)
+		(fields_autoplaced yes)
+		(effects
+			(font
+				(size 1.27 1.27)
+			)
+			(justify left)
+		)
+	)
+	(hierarchical_label "INTVCC"
+		(shape output)
+		(at 24.13 66.04 180)
+		(fields_autoplaced yes)
+		(effects
+			(font
+				(size 1.27 1.27)
+			)
+			(justify right)
+		)
+	)
 	(hierarchical_label "GATE1"
 		(shape output)
@@
 		)
 	)
+	(hierarchical_label "SHDN"
+		(shape output)
+		(at 77.47 66.04 0)
+		(fields_autoplaced yes)
+		(effects
+			(font
+				(size 1.27 1.27)
+			)
+			(justify left)
+		)
+	)
 	(hierarchical_label "SOURCE1"
 		(shape input)
@@
 		(on_board yes)
 		(dnp no)
-		(property "Reference" "CINTV_CC1"
+		(property "Reference" "CINTVCC1"
 			(at 13.462 70.104 0)
 			(effects
@@
 			(project "Power-Secondary"
 				(path "/ba21eba1-72a9-489c-9498-a38516b9f252/3184e9c2-8c00-4ca3-a214-8a04df6b61e9"
-					(reference "CINTV_CC1")
+					(reference "CINTVCC1")
 					(unit 1)
 				)
@@
 					(unit 1)
 				)
+			)
+		)
+	)
+	(symbol
+		(lib_id "power:PWR_FLAG")
+		(at 29.21 68.58 180)
+		(unit 1)
+		(exclude_from_sim no)
+		(in_bom yes)
+		(on_board yes)
+		(dnp no)
+		(fields_autoplaced yes)
+		(property "Reference" "#FLG04"
+			(at 29.21 70.485 0)
+			(effects
+				(font
+					(size 1.27 1.27)
+				)
+				(hide yes)
+			)
+		)
+		(property "Value" "PWR_FLAG"
+			(at 29.21 73.66 0)
+			(effects
+				(font
+					(size 1.27 1.27)
+				)
+				(hide yes)
+			)
+		)
+		(property "Footprint" ""
+			(at 29.21 68.58 0)
+			(effects
+				(font
+					(size 1.27 1.27)
+				)
+				(hide yes)
+			)
+		)
+		(property "Datasheet" "~"
+			(at 29.21 68.58 0)
+			(effects
+				(font
+					(size 1.27 1.27)
+				)
+				(hide yes)
+			)
+		)
+		(property "Description" "Special symbol for telling ERC where power comes from"
+			(at 29.21 68.58 0)
+			(effects
+				(font
+					(size 1.27 1.27)
+				)
+				(hide yes)
+			)
+		)
+		(pin "1"
+		)
+		(instances
+			(project "Power-Secondary"
+				(path "/ba21eba1-72a9-489c-9498-a38516b9f252/3184e9c2-8c00-4ca3-a214-8a04df6b61e9"
+					(reference "#FLG04")
+					(unit 1)
+				)

Commit message: final footprint assignments
Parts:
- CTMR1, CTMR2: footprint (none) -> Capacitor_SMD:C_0805_2012Metric
Changed lines of the file:
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@@
 			)
 		)
-		(property "Footprint" ""
+		(property "Footprint" "Capacitor_SMD:C_0805_2012Metric"
 			(at 141.9352 182.88 0)
 			(effects
@@
 			)
 		)
-		(property "Footprint" ""
+		(property "Footprint" "Capacitor_SMD:C_0805_2012Metric"
 			(at 160.9852 182.88 0)
 			(effects
